Commit message: added in forearm

File: robot/humanoid/flo_humanoid/urdf/flo.urdf.xacro (robot description, xacro)
@@ -1,16 +1,59 @@
 <?xml version="1.0"?>
 <robot name="lilFlo"  xmlns:xacro="http://ros.org/wiki/xacro">
-  <xacro:macro name="default_inertial" params="mass">
-    <inertial>
-      <mass value="${mass}" />
-      <inertia ixx="1.0" ixy="0.0" ixz="0.0" iyy="1.0" iyz="0.0" izz="1.0" />
-    </inertial>
-  </xacro:macro>
-  <link name="base_link">
-    <visual>
-      <geometry>
-        <mesh filename="file://$(arg mesh_dir)BODY - FLO-CHEST-01.stl"/>
-      </geometry>
-    </visual>
-  </link>
+    <xacro:property name="mesh_extension" value="dae" />
+    <xacro:macro name="add_mesh" params="file_name xyz:='0 0 0' rpy:='0 0 0'">
+        <visual>
+            <origin xyz="${xyz}" rpy="${rpy}"/>
+            <geometry>
+                <mesh filename="file://$(arg mesh_dir)${file_name}.${mesh_extension}"/>
+            </geometry>
+        </visual>
+    </xacro:macro>
+    <xacro:macro name="default_inertial" params="mass">
+        <inertial>
+            <mass value="${mass}" />
+            <inertia ixx="1.0" ixy="0.0" ixz="0.0" iyy="1.0" iyz="0.0" izz="1.0" />
+        </inertial>
+    </xacro:macro>
+    <link name="base_link"/>
+    <link name="hang_bar">
+        <visual>
+            <origin rpy="0 ${pi/2} 0"/>
+            <geometry>
+                <cylinder length=".046" radius="0.0029972"/>
+            </geometry>
+        </visual>
+    </link>
+    <joint name="bar2base" type="fixed">
+        <parent link="base_link"/>
+        <child link="hang_bar"/>
+        <!-- <origin rpy="0 ${pi/2} ${pi}" xyz="0 0 0"/> -->
+    </joint>
+    <link name="chest">
+        <xacro:add_mesh file_name="BODY - FLO-CHEST-01"/>
+    </link>
+    <joint name="chest_ref" type="fixed">
+        <parent link="hang_bar"/>
+        <child link="chest"/>
+        <origin xyz=".0435 -.0720 .0466"/>
+    </joint>
+    <link name="left_shoulder">
+        <xacro:add_mesh file_name="FLO-ARM-01 UPPER ARM MOUNT - FLO-ARM-LEFT-01 UPPER ARM MOUNT" rpy="0 ${pi/2} 0"/>
+    </link>
+    <joint name="left_shoulder_flexionextension" type="revolute">
+        <axis xyz="0 0 1"/>
+        <limit effort="1000.0" lower="0.0" upper="2.5" velocity="0.5"/>
+        <parent link="hang_bar"/>
+        <child link="left_shoulder"/>
+        <origin xyz="-0.04965 .072  -.02153" rpy="${pi/2} 0 ${-pi/2}"/>
+    </joint>
+    <link name="left_forearm">
+    </link>
+    <joint name="lef_shoulder_abduction" type="revolute">
+        <axis xyz="0 0 1"/>
+        <limit effort="1000.0" lower="0.0" upper="2.5" velocity="0.5"/>
+        <parent link="left_shoulder"/>
+        <child link="left_forearm"/>
+        <origin xyz="0 0 .04572" rpy="0 ${-pi/2} 0"/>
+    </joint>
 </robot>

Commit message: finished left arm

File: robot/humanoid/flo_humanoid/urdf/flo.urdf.xacro (robot description, xacro)
@@ -36,5 +36,5 @@
         <parent link="hang_bar"/>
         <child link="chest"/>
-        <origin xyz=".0435 -.0720 .0466"/>
+        <origin xyz="-0.04660000 .0720 -0.04351694" rpy="0 ${pi/2} ${pi}"/>
     </joint>
     <link name="left_shoulder">
@@ -48,12 +48,33 @@
         <origin xyz="-0.04965 .072  -.02153" rpy="${pi/2} 0 ${-pi/2}"/>
     </joint>
-    <link name="left_forearm">
+    <link name="left_upperarm">
+        <xacro:add_mesh file_name="FLO-ARM-02 MIDDLE ARM DOUBLE MOUNT-LEFT" xyz="-0.00250 -0.04318000 000" rpy="${-pi/2} ${pi/2} 0"/>
     </link>
-    <joint name="lef_shoulder_abduction" type="revolute">
+    <joint name="left_shoulder_abduction" type="revolute">
         <axis xyz="0 0 1"/>
         <limit effort="1000.0" lower="0.0" upper="2.5" velocity="0.5"/>
         <parent link="left_shoulder"/>
-        <child link="left_forearm"/>
+        <child link="left_upperarm"/>
         <origin xyz="0 0 .04572" rpy="0 ${-pi/2} 0"/>
     </joint>
+    <link name="left_elbow">
+        <xacro:add_mesh file_name="FLO-ARM-04 MID ARM CONNECTOR - FLO-ARM-LEFT-04 MID ARM CONNECTOR" rpy="0 ${pi/2} ${pi/2}"/>
+    </link>
+    <joint name="left_shoulder_rotation" type="revolute">
+        <axis xyz="0 0 1"/>
+        <limit effort="1000.0" lower="0.0" upper="2.5" velocity="0.5"/>
+        <parent link="left_upperarm"/>
+        <child link="left_elbow"/>
+        <origin xyz="0.07951 0 0" rpy="0 ${pi/2} 0"/>
+    </joint>
+    <link name="left_forearm">
+        <xacro:add_mesh file_name="FLO LOWER ARM - LEFT" xyz="0.01071292 0 0" rpy="${pi} 0 0"/>
+    </link>
+    <joint name="left_elbow_flexion" type="revolute">
+        <axis xyz="0 0 1"/>
+        <limit effort="1000.0" lower="0.0" upper="2.5" velocity="0.5"/>
+        <parent link="left_elbow"/>
+        <child link="left_forearm"/>
+        <origin xyz="0 0 0.03442" rpy="0 ${-pi/2} 0"/>
+    </joint>
 </robot>

Commit message: changed the name of the elbow fexextension

File: robot/humanoid/flo_humanoid/urdf/flo.urdf.xacro (robot description, xacro)
@@ -71,5 +71,5 @@
         <xacro:add_mesh file_name="FLO LOWER ARM - LEFT" xyz="0.01071292 0 0" rpy="${pi} 0 0"/>
     </link>
-    <joint name="left_elbow_flexion" type="revolute">
+    <joint name="left_elbow_flexionextension" type="revolute">
         <axis xyz="0 0 1"/>
         <limit effort="1000.0" lower="0.0" upper="2.5" velocity="0.5"/>

Commit message: got a workable version of right arm in urdf

File: robot/humanoid/flo_humanoid/urdf/flo.urdf.xacro (robot description, xacro)
@@ -1,4 +1,5 @@
 <?xml version="1.0"?>
 <robot name="lilFlo"  xmlns:xacro="http://ros.org/wiki/xacro">
+    <!--Macros-->
     <xacro:property name="mesh_extension" value="dae" />
     <xacro:macro name="add_mesh" params="file_name xyz:='0 0 0' rpy:='0 0 0'">
@@ -16,4 +17,5 @@
         </inertial>
     </xacro:macro>
+    <!--Core of robot-->
     <link name="base_link"/>
     <link name="hang_bar">
@@ -30,4 +32,5 @@
         <!-- <origin rpy="0 ${pi/2} ${pi}" xyz="0 0 0"/> -->
     </joint>
+    <!--chest-->
     <link name="chest">
         <xacro:add_mesh file_name="BODY - FLO-CHEST-01"/>
@@ -38,4 +41,5 @@
         <origin xyz="-0.04660000 .0720 -0.04351694" rpy="0 ${pi/2} ${pi}"/>
     </joint>
+    <!--Left Arm-->
     <link name="left_shoulder">
         <xacro:add_mesh file_name="FLO-ARM-01 UPPER ARM MOUNT - FLO-ARM-LEFT-01 UPPER ARM MOUNT" rpy="0 ${pi/2} 0"/>
@@ -78,3 +82,44 @@
         <origin xyz="0 0 0.03442" rpy="0 ${-pi/2} 0"/>
     </joint>
+    <!--Right Arm-->
+    <link name="right_shoulder">
+        <xacro:add_mesh file_name="FLO-ARM-01 UPPER ARM MOUNT - FLO-ARM-RIGHT-01 UPPER ARM MOUNT" rpy="0 ${pi/2} 0"/>
+    </link>
+    <joint name="right_shoulder_flexionextension" type="revolute">
+        <axis xyz="0 0 1"/>
+        <limit effort="1000.0" lower="0.0" upper="2.5" velocity="0.5"/>
+        <parent link="hang_bar"/>
+        <child link="right_shoulder"/>
+        <origin xyz="0.04965 .072  -.02153" rpy="${pi/2} 0 ${-pi/2}"/>
+    </joint>
+    <link name="right_upperarm">
+        <xacro:add_mesh file_name="FLO-ARM-02 MIDDLE ARM DOUBLE MOUNT-RIGHT" xyz="0.00250 -0.04318000 000" rpy="${pi/2} ${pi/2} 0"/>
+    </link>
+    <joint name="right_shoulder_abduction" type="revolute">
+        <axis xyz="0 0 -1"/>
+        <limit effort="1000.0" lower="0.0" upper="2.5" velocity="0.5"/>
+        <parent link="right_shoulder"/>
+        <child link="right_upperarm"/>
+        <origin xyz="0 0 -.04572" rpy="0 ${-pi/2} 0"/>
+    </joint>
+    <link name="right_elbow">
+        <xacro:add_mesh file_name="FLO-ARM-04 MID ARM CONNECTOR - FLO-ARM-RIGHT-04 MID ARM CONNECTOR" rpy="0 ${pi/2} ${pi/2}"/>
+    </link>
+    <joint name="right_shoulder_rotation" type="revolute">
+        <axis xyz="0 0 1"/>
+        <limit effort="1000.0" lower="0.0" upper="2.5" velocity="0.5"/>
+        <parent link="right_upperarm"/>
+        <child link="right_elbow"/>
+        <origin xyz="-0.07951 0 0" rpy="0 ${pi/2} 0"/>
+    </joint>
+    <link name="right_forearm">
+        <xacro:add_mesh file_name="FLO LOWER ARM - RIGHT" xyz="-0.01071292 0 0.11378887" rpy="${pi} ${pi} 0"/>
+    </link>
+    <joint name="right_elbow_flexionextension" type="revolute">
+        <axis xyz="0 0 -1"/>
+        <limit effort="1000.0" lower="0.0" upper="2.5" velocity="0.5"/>
+        <parent link="right_elbow"/>
+        <child link="right_forearm"/>
+        <origin xyz="0 0 -0.03442" rpy="0 ${-pi/2} 0"/>
+    </joint>
 </robot>

Commit message: changed urdf to have a more logical neutral pose

File: robot/humanoid/flo_humanoid/urdf/flo.urdf.xacro (robot description, xacro)
@@ -60,5 +60,5 @@
         <parent link="left_shoulder"/>
         <child link="left_upperarm"/>
-        <origin xyz="0 0 .04572" rpy="0 ${-pi/2} 0"/>
+        <origin xyz="0 0 .04572" rpy="${pi/2} 0 ${-pi/2}"/>
     </joint>
     <link name="left_elbow">
@@ -70,5 +70,5 @@
         <parent link="left_upperarm"/>
         <child link="left_elbow"/>
-        <origin xyz="0.07951 0 0" rpy="0 ${pi/2} 0"/>
+        <origin xyz="0.07951 0 0" rpy="${pi/2} 0 ${pi/2}"/>
     </joint>
     <link name="left_forearm">
@@ -101,5 +101,5 @@
         <parent link="right_shoulder"/>
         <child link="right_upperarm"/>
-        <origin xyz="0 0 -.04572" rpy="0 ${-pi/2} 0"/>
+        <origin xyz="0 0 -.04572" rpy="${pi/2} 0 ${pi/2}"/>
     </joint>
     <link name="right_elbow">
@@ -111,5 +111,5 @@
         <parent link="right_upperarm"/>
         <child link="right_elbow"/>
-        <origin xyz="-0.07951 0 0" rpy="0 ${pi/2} 0"/>
+        <origin xyz="-0.07951 0 0" rpy="${-pi/2} 0 ${-pi/2}"/>
     </joint>
     <link name="right_forearm">

Commit message: fixed the orientation of joints

File: robot/humanoid/flo_humanoid/urdf/flo.urdf.xacro (robot description, xacro)
@@ -46,5 +46,5 @@
     </link>
     <joint name="left_shoulder_flexionextension" type="revolute">
-        <axis xyz="0 0 1"/>
+        <axis xyz="0 0 -1"/>
         <limit effort="1000.0" lower="0.0" upper="2.5" velocity="0.5"/>
         <parent link="hang_bar"/>
@@ -87,5 +87,5 @@
     </link>
     <joint name="right_shoulder_flexionextension" type="revolute">
-        <axis xyz="0 0 1"/>
+        <axis xyz="0 0 -1"/>
         <limit effort="1000.0" lower="0.0" upper="2.5" velocity="0.5"/>
         <parent link="hang_bar"/>
@@ -101,5 +101,5 @@
         <parent link="right_shoulder"/>
         <child link="right_upperarm"/>
-        <origin xyz="0 0 -.04572" rpy="${pi/2} 0 ${pi/2}"/>
+        <origin xyz="0 0 -.04572" rpy="${-pi/2} 0 ${pi/2}"/>
     </joint>
     <link name="right_elbow">
@@ -111,5 +111,5 @@
         <parent link="right_upperarm"/>
         <child link="right_elbow"/>
-        <origin xyz="-0.07951 0 0" rpy="${-pi/2} 0 ${-pi/2}"/>
+        <origin xyz="-0.07951 0 0" rpy="${pi/2} 0 ${pi/2}"/>
     </joint>
     <link name="right_forearm">
