Commit message: got launch files working across the two computers

File: flo_humanoid/urdf/flo.urdf.xacro (robot description, xacro)
@@ -7,5 +7,5 @@
             <origin xyz="${xyz}" rpy="${rpy}"/>
             <geometry>
-                <mesh filename="file://$(arg mesh_dir)${file_name}.${mesh_extension}"/>
+                <mesh filename="package://flo_humanoid/urdf/CAD_refs/${file_name}.${mesh_extension}"/>
             </geometry>
         </visual>

Commit message: Flipped axes for roation of shoulders
I don't understand why this was needed, but the shoulders were moving in
the opposit direction of reality in URDF displays. Having to make this
change worries me since it was working before. More testing is needed.

File: flo_humanoid/urdf/flo.urdf.xacro (robot description, xacro)
@@ -46,5 +46,5 @@
     </link>
     <joint name="left_shoulder_flexionextension" type="revolute">
-        <axis xyz="0 0 -1"/>
+        <axis xyz="0 0 1"/>
         <limit effort="1000.0" lower="0.0" upper="2.5" velocity="0.5"/>
         <parent link="hang_bar"/>
@@ -87,5 +87,5 @@
     </link>
     <joint name="right_shoulder_flexionextension" type="revolute">
-        <axis xyz="0 0 -1"/>
+        <axis xyz="0 0 1"/>
         <limit effort="1000.0" lower="0.0" upper="2.5" velocity="0.5"/>
         <parent link="hang_bar"/>
